File: hardware/right_hand_4x2/switches.kicad_sch (KiCad schematic)
At the start: 16 parts, among them SW1 SW_SPST, SW2 SW_SPST, SW3 SW_SPST, SW4 SW_SPST, SW5 SW_SPST, SW6 SW_SPST, SW7 SW_SPST, SW8 SW_SPST

Commit message: replaced diodes with easier to solder part
Parts:
- removed D1, D2, D3, D4, D5, D6, D7, D8: 1N4148WS, Diode_SMD:D_SOD-323, symbol Diode:1N4148WS
- added D1, D2, D3, D4, D5, D6, D7, D8: 1N4148W, Diode_SMD:D_SOD-123, symbol Diode:1N4148W
Connections:
- net row0: now also D1.1 (K), D2.1 (K), D3.1 (K), D4.1 (K)
- net row1: now also D5.1 (K), D6.1 (K), D7.1 (K), D8.1 (K)
- net at SW1.2 (B): now also D1.2 (A)
- net at SW8.2 (B): now also D8.2 (A)
- net at SW4.2 (B): now also D4.2 (A)
- net at SW6.2 (B): now also D6.2 (A)
- net at SW2.2 (B): now also D2.2 (A)
- net at SW7.2 (B): now also D7.2 (A)
- net at SW5.2 (B): now also D5.2 (A)
- net at SW3.2 (B): now also D3.2 (A)
