File: hardware/right_hand_4x2/right_hand_4x2.kicad_sch (KiCad schematic)
At the start: 0 parts

Commit message: Layout udpate
Parts:
- added H1, H2, H3, H4: MountingHole_Pad, MountingHole:MountingHole_3.2mm_M3_Pad, symbol Mechanical:MountingHole_Pad
Other:
- note added: "M3 Mounting Holes"

Commit message: layout update
Parts:
- H1, H2, H3, H4: footprint MountingHole:MountingHole_3.2mm_M3_Pad -> MountingHole:MountingHole_3.2mm_M3_ISO7380_Pad_TopOnly
Connections:
- net GND: now reaches H2.1
- net GND: now also H1.1, H3.1, H4.1
Other:
- moved on the sheet: H3, H4
