File: hardware/right_hand_4x2/right_hand_4x2.kicad_pcb (KiCad board)
At the start: 2 copper layers, 117 x 50 mm, 34 parts, among them SW1 SW_SPST, SW2 SW_SPST, SW3 SW_SPST, SW4 SW_SPST, SW5 SW_SPST, SW6 SW_SPST, SW7 SW_SPST, SW8 SW_SPST, U1 RP2040-ZERO

Commit message: Layout udpate
Parts:
- added H1: MountingHole_Pad, MountingHole:MountingHole_3.2mm_M3_Pad, F.Cu at (99.4, 49.5)
- added H2: MountingHole_Pad, MountingHole:MountingHole_3.2mm_M3_Pad, F.Cu at (207.8, 49.2)
- added H3: MountingHole_Pad, MountingHole:MountingHole_3.2mm_M3_Pad, F.Cu at (99.5, 91.0)
- added H4: MountingHole_Pad, MountingHole:MountingHole_3.2mm_M3_Pad, F.Cu at (207.9, 91.0)
- moved C5 6.33 mm to (105.6, 92.1), turned to 180 degrees
- moved U1 5.83 mm to (194.1, 58.5)
- moved D10 5.11 mm to (113.0, 65.1)
- moved SW5 5.09 mm to (115.3, 75.0)
- moved C1 5.00 mm to (104.6, 66.9)
- moved SW1 5.00 mm to (115.3, 50.0)
- moved D14 4.96 mm to (112.5, 90.2)
- moved D4 4.92 mm to (167.8, 58.0), turned to 90 degrees
- moved D8 4.87 mm to (168.0, 83.1), turned to 90 degrees
- moved R1 3.30 mm to (193.2, 74.2)
- moved C6 3.29 mm to (125.0, 91.8), turned to 180 degrees
- moved SW8 3.14 mm to (175.3, 75.0)
- moved D17 3.04 mm to (173.1, 90.3)
- moved D5 2.96 mm to (108.1, 82.9), turned to 90 degrees
- moved D1 2.92 mm to (108.0, 58.1), turned to 90 degrees
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Other:
- board size 117 x 50 mm -> 119 x 50 mm

Commit message: replaced diodes with easier to solder part
Parts:
- D1, D2, D3, D4, D5, D6, D7, D8: value 1N4148WS -> 1N4148W; footprint Diode_SMD:D_SOD-323 -> Diode_SMD:D_SOD-123
- moved D1 2.16 mm to (105.9, 58.6)
- moved D2 2.14 mm to (126.1, 58.6)
- moved D7 2.11 mm to (146.1, 83.3)
- moved D6 1.94 mm to (126.3, 83.3)
- moved D4 1.91 mm to (166.0, 58.6)
- moved D8 1.91 mm to (166.1, 83.3)
- moved D5 1.71 mm to (106.4, 83.1)
- moved D3 1.66 mm to (146.3, 58.6)
- moved C5 1.51 mm to (106.7, 91.1)
- moved D14 0.91 mm to (113.5, 90.2)
Routing:
- net col0: track 0.00 -> 88.4 mm
- net col1: track 0.00 -> 68.7 mm
- net col2: track 0.00 -> 48.9 mm
- net row1: track 0.00 -> 21.3 mm

Commit message: layout update
Parts:
- H1, H2, H3, H4: footprint MountingHole:MountingHole_3.2mm_M3_Pad -> MountingHole:MountingHole_3.2mm_M3_ISO7380_Pad_TopOnly; moved to B.Cu
- moved R1 1.00 mm to (193.1, 75.2)
- turned H1 to 0 degrees
- turned H2 to 0 degrees
- turned H3 to 180 degrees
- turned H4 to 180 degrees
Connections:
- H1 pad 1: unconnected-(H1-Pad1) -> GND
- H2 pad 1: unconnected-(H2-Pad1) -> GND
- H3 pad 1: unconnected-(H3-Pad1) -> GND
- H4 pad 1: unconnected-(H4-Pad1) -> GND
Routing:
- net +5V: track 0.00 -> 182.6 mm, vias 0 -> 1
- net row1: track 21.3 -> 122.0 mm, vias 0 -> 1
- net row0: track 0.00 -> 96.5 mm
- net rgb: track 0.00 -> 83.4 mm, vias 0 -> 1
- net col0: track 88.4 -> 137.2 mm
- net col4: track 0.00 -> 34.9 mm
- net Net-(D11-DOUT): track 0.00 -> 30.4 mm
- net Net-(D15-DOUT): track 0.00 -> 30.3 mm
- net Net-(D12-DOUT): track 0.00 -> 29.9 mm
- net Net-(D16-DOUT): track 0.00 -> 29.7 mm
- net Net-(D10-DOUT): track 0.00 -> 29.6 mm
- net Net-(D14-DOUT): track 0.00 -> 28.2 mm
- net col1: track 68.7 -> 96.0 mm, vias 0 -> 2
- net col2: track 48.9 -> 76.2 mm, vias 0 -> 2
- net Net-(U1-GP11): track 0.00 -> 6.56 mm
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
Commit message: layout completed v1
Routing:
- net GND: track 0.00 -> 383.5 mm, vias 0 -> 11
- net Net-(D13-DOUT): track 0.00 -> 98.2 mm
- net +5V: track 182.6 -> 221.5 mm
- net rgb: track 83.4 -> 84.7 mm
- net row0: track 96.5 -> 97.0 mm, vias 0 -> 1
- added copper zone on B.Cu, net GND
- added copper zone on F.Cu, net GND

Commit message: layout rev0.1 done, gerber files gen
Other:
- board text added: "CAD stands for Computer-aided design"
- board text added: "REV: 0.1 // DATE: AUG 2026"
- board text added: "Ψ *"
- board text added: "Ψ ★"
- board text added: "Ψ 🗲 ★"
- board text added: "キーパッド"
Changed lines of the file:
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@@
 			(outputformat 1)
 			(mirror no)
-			(drillshape 1)
+			(drillshape 0)
 			(scaleselection 1)
-			(outputdirectory "")
+			(outputdirectory "fab-files/")
 		)
 	)
@@
 	)
 	(gr_rect
+		(start 111.93125 86.925)
+		(end 151.76875 93.575)
+		(stroke
+			(width 0.1)
+			(type solid)
+		)
+		(fill yes)
+		(layer "B.SilkS")
+	)
+	(gr_rect
+		(start 180.43125 76.7125)
+		(end 201.7 87.55)
+		(stroke
+			(width 0.1)
+			(type solid)
+		)
+		(fill yes)
+		(layer "B.SilkS")
+	)
+	(gr_rect
 		(start 94 45)
 		(end 213 95)
@@
 	)
 	(gr_text " _   _\n *   *\n   |\n\\_____/"
-		(at 185.5 92.1 0)
+		(at 185.55 90.25 0)
 		(layer "F.SilkS")
 		(effects
 			(font
 				(size 3 3)
-				(thickness 0.2)
+				(thickness 0.508)
+				(bold yes)
 			)
 			(justify left bottom)
 		)
 	)
+	(gr_text "Ψ\n*"
+		(at 209.25 65.65 0)
+		(layer "F.SilkS")
+		(effects
+			(font
+				(face "Ubuntu Sans Mono")
+				(size 3.048 3.048)
+				(thickness 0.127)
+			)
+			(justify left bottom mirror)
+		)
+		(render_cache "Ψ\n*" 0
+			(polygon
+				(pts
+					(xy 208.212978 60.0112) (xy 208.212978 59.23883) (xy 208.4126 59.222601) (xy 208.570274 59.172343)
+					(xy 208.695196 59.091615) (xy 208.797788 58.981039) (xy 208.88125 58.841371) (xy 208.94496 58.667091)
+					(xy 208.999901 58.383203) (xy 209.019592 58.043985) (xy 209.019592 57.054049) (xy 208.648296 57.054049)
+					(xy 208.648296 58.005645) (xy 208.637578 58.319042) (xy 208.609957 58.541093) (xy 208.574951 58.676022)
+					(xy 208.530184 58.774378) (xy 208.47763 58.844085) (xy 208.409389 58.895888) (xy 208.322952 58.928397)
+					(xy 208.212978 58.940119) (xy 208.212978 57.740993) (xy 207.89733 57.740993) (xy 207.89733 58.940119)
+					(xy 207.787481 58.928402) (xy 207.701101 58.895897) (xy 207.632863 58.844085) (xy 207.580218 58.774358)
+					(xy 207.535449 58.676001) (xy 207.500537 58.541093) (xy 207.472782 58.319042) (xy 207.462011 58.005645)
+					(xy 207.462011 57.054049) (xy 207.090716 57.054049) (xy 207.090716 58.043985) (xy 207.109349 58.383392)
+					(xy 207.161253 58.667091) (xy 207.222373 58.841294) (xy 207.304346 58.980934) (xy 207.40655 59.091615)
+					(xy 207.531618 59.172007) (xy 207.691864 59.222433) (xy 207.89733 59.23883) (xy 207.89733 60.0112)
+				)
+			)
+			(polygon
+				(pts
+					(xy 208.43501 63.902935) (xy 208.729441 63.685183) (xy 208.631174 63.561418) (xy 208.499033 63.407874)
+					(xy 208.358146 63.26494) (xy 208.212978 63.126285) (xy 208.40728 63.096507) (xy 208.599348 63.064496)
+					(xy 208.789184 63.019643) (xy 208.96413 62.968461) (xy 208.853206 62.622663) (xy 208.67826 62.690967)
+					(xy 208.4968 62.765784) (xy 208.321854 62.846743) (xy 208.149141 62.934217) (xy 208.189713 62.708089)
+					(xy 208.221725 62.484195) (xy 208.234381 62.255835) (xy 208.234381 62.174689) (xy 207.867366 62.174689)
+					(xy 207.867366 62.259929) (xy 207.880207 62.486243) (xy 207.912219 62.708089) (xy 207.952792 62.934217)
+					(xy 207.765003 62.838182) (xy 207.577402 62.750709) (xy 207.389427 62.673844) (xy 207.265662 62.626944)
+					(xy 207.150458 62.972556) (xy 207.282785 63.006801) (xy 207.436514 63.041046) (xy 207.590057 63.072871)
+					(xy 207.743787 63.098554) (xy 207.89733 63.122005) (xy 207.737273 63.26922) (xy 207.585777 63.418669)
+					(xy 207.45345 63.582821) (xy 207.381052 63.689463) (xy 207.688139 63.902935) (xy 207.765003 63.787731)
+					(xy 207.869599 63.608504) (xy 207.961353 63.427044) (xy 208.050873 63.24577) (xy 208.14486 63.433558)
+					(xy 208.240895 63.619113) (xy 208.358146 63.800387)
+				)
+			)
+		)
+	)
+	(gr_text "REV: 0.1 // DATE: AUG 2026"
+		(at 187.25 92.85 0)
+		(layer "B.SilkS")
+		(effects
+			(font
+				(size 1.524 1.524)
+				(thickness 0.254)
+			)
+			(justify left bottom mirror)
+		)
+	)
+	(gr_text "CAD stands for Computer-aided design"
+		(at 182.05 69.85 0)
+		(layer "B.SilkS")
+		(effects
+			(font
+				(size 2.286 2.286)
+				(thickness 0.381)
+				(bold yes)
+			)
+			(justify left bottom mirror)
+		)
+	)
+	(gr_text "キーパッド"
+		(at 100.35 63.85 90)
+		(layer "B.SilkS")
+		(effects
+			(font
+				(size 2.286 2.286)
+				(thickness 0.381)
+			)
+			(justify left bottom mirror)
+		)
+	)
+	(gr_text "Ψ 🗲 ★"
+		(at 159.25 112.35 0)
+		(layer "B.SilkS")
+		(effects
+			(font
+				(face "Bitstream Charter")
+				(size 1 1)
+				(thickness 0.1)
+			)
+			(justify left bottom mirror)
+		)
+		(render_cache "Ψ 🗲 ★" 0)
+	)
+	(gr_text "Ψ ★"
+		(at 168.5 114.6 0)
+		(layer "B.SilkS")
+		(effects
+			(font
+				(face "D050000L")
+				(size 1 1)
+				(thickness 0.1)
+			)
+			(justify left bottom mirror)
+		)
+		(render_cache "Ψ ★" 0)
+	)
+	(gr_text "Ψ\n*"
+		(at 209.1 65.15 0)
+		(layer "B.SilkS")
+		(effects
+			(font
+				(face "Ubuntu Sans Mono")
+				(size 3.048 3.048)
+				(thickness 0.127)
+			)
+			(justify left bottom mirror)
+		)
+		(render_cache "Ψ\n*" 0
+			(polygon
+				(pts
+					(xy 208.062978 59.5112) (xy 208.062978 58.73883) (xy 208.2626 58.722601) (xy 208.420274 58.672343)
+					(xy 208.545196 58.591615) (xy 208.647788 58.481039) (xy 208.73125 58.341371) (xy 208.79496 58.167091)
+					(xy 208.849901 57.883203) (xy 208.869592 57.543985) (xy 208.869592 56.554049) (xy 208.498296 56.554049)
+					(xy 208.498296 57.505645) (xy 208.487578 57.819042) (xy 208.459957 58.041093) (xy 208.424951 58.176022)
+					(xy 208.380184 58.274378) (xy 208.32763 58.344085) (xy 208.259389 58.395888) (xy 208.172952 58.428397)
+					(xy 208.062978 58.440119) (xy 208.062978 57.240993) (xy 207.74733 57.240993) (xy 207.74733 58.440119)
+					(xy 207.637481 58.428402) (xy 207.551101 58.395897) (xy 207.482863 58.344085) (xy 207.430218 58.274358)
+					(xy 207.385449 58.176001) (xy 207.350537 58.041093) (xy 207.322782 57.819042) (xy 207.312011 57.505645)
+					(xy 207.312011 56.554049) (xy 206.940716 56.554049) (xy 206.940716 57.543985) (xy 206.959349 57.883392)
+					(xy 207.011253 58.167091) (xy 207.072373 58.341294) (xy 207.154346 58.480934) (xy 207.25655 58.591615)
+					(xy 207.381618 58.672007) (xy 207.541864 58.722433) (xy 207.74733 58.73883) (xy 207.74733 59.5112)
+				)
+			)
+			(polygon
+				(pts
+					(xy 208.28501 63.402935) (xy 208.579441 63.185183) (xy 208.481174 63.061418) (xy 208.349033 62.907874)
+					(xy 208.208146 62.76494) (xy 208.062978 62.626285) (xy 208.25728 62.596507) (xy 208.449348 62.564496)
+					(xy 208.639184 62.519643) (xy 208.81413 62.468461) (xy 208.703206 62.122663) (xy 208.52826 62.190967)
+					(xy 208.3468 62.265784) (xy 208.171854 62.346743) (xy 207.999141 62.434217) (xy 208.039713 62.208089)
+					(xy 208.071725 61.984195) (xy 208.084381 61.755835) (xy 208.084381 61.674689) (xy 207.717366 61.674689)
+					(xy 207.717366 61.759929) (xy 207.730207 61.986243) (xy 207.762219 62.208089) (xy 207.802792 62.434217)
+					(xy 207.615003 62.338182) (xy 207.427402 62.250709) (xy 207.239427 62.173844) (xy 207.115662 62.126944)
+					(xy 207.000458 62.472556) (xy 207.132785 62.506801) (xy 207.286514 62.541046) (xy 207.440057 62.572871)
+					(xy 207.593787 62.598554) (xy 207.74733 62.622005) (xy 207.587273 62.76922) (xy 207.435777 62.918669)
+					(xy 207.30345 63.082821) (xy 207.231052 63.189463) (xy 207.538139 63.402935) (xy 207.615003 63.287731)
+					(xy 207.719599 63.108504) (xy 207.811353 62.927044) (xy 207.900873 62.74577) (xy 207.99486 62.933558)
+					(xy 208.090895 63.119113) (xy 208.208146 63.300387)
+				)
+			)
+		)
+	)
